File: Layout/68EC020TK-V02.sch (EAGLE design)
At the start: 100 parts, among them IC10 74HCT245PW, IC11 74HCT245PW, IC12 AM29F010S, IC13 XC95288XL-TQ144, IC14 ICS570B, IC15 74HCT245PW, IC2 MC68EC020RP, IC3 74ACT16245, IC4 74ACT16245, IC5 LD117AS33TR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

Commit message: fixed parts but mem cfg not bug free
Parts:
- C24, C25, C26, C27, C28, C29, C30, C31: value 10nF -> 100nF
- C39: value 47µF -> 47uF; device rcl:C-EUC0805K -> rcl:C-EUC1206K
- C43, C44: value (none) -> 100nF
- FB1: value 100Ohm@100MHz -> 120Ohm@100MHz 0.5A
- IC12: value AM29F010S -> AM29F010S-10
- IC13: value XC95288XL-TQ144 -> XC95288XL-TQ144-10ns
- IC6, IC7: value 74ALVT16543 -> 74LVT16543
- IC8, IC9: value K4S56163 -> AS4C4M16SA-6TCN
- X1: value (none) -> 16,66MHz / 3.3V
Changed lines of the file:
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@@
 <part name="GND8" library="supply1" deviceset="GND" device="" value="GND"/>
 <part name="P+8" library="supply1" deviceset="3,3V" device="" value="3,3V"/>
-<part name="IC8" library="SMD-IC" deviceset="K4S56163@2" device="" value="K4S56163"/>
-<part name="IC9" library="SMD-IC" deviceset="K4S56163@2" device="" value="K4S56163"/>
+<part name="IC8" library="SMD-IC" deviceset="K4S56163@2" device="" value="AS4C4M16SA-6TCN"/>
+<part name="IC9" library="SMD-IC" deviceset="K4S56163@2" device="" value="AS4C4M16SA-6TCN"/>
 <part name="C17" library="rcl" deviceset="C-EU" device="C0603K" value="100nF"/>
 <part name="C18" library="rcl" deviceset="C-EU" device="C0603K" value="100nF"/>
@@
 <part name="GND11" library="supply1" deviceset="GND" device="" value="GND"/>
 <part name="GND12" library="supply1" deviceset="GND" device="" value="GND"/>
-<part name="IC6" library="SMD-IC" deviceset="ABT16543@2" device="" value="74ALVT16543"/>
-<part name="IC7" library="SMD-IC" deviceset="ABT16543@2" device="" value="74ALVT16543"/>
+<part name="IC6" library="SMD-IC" deviceset="ABT16543@2" device="" value="74LVT16543"/>
+<part name="IC7" library="SMD-IC" deviceset="ABT16543@2" device="" value="74LVT16543"/>
 <part name="RN1" library="SMD" deviceset="R-NETZ@3" device="" value="33R"/>
 <part name="RN2" library="SMD" deviceset="R-NETZ@3" device="" value="33R"/>
@@
 <part name="RN5" library="SMD" deviceset="R-NETZ@3" device="" value="33R"/>
 <part name="RN6" library="SMD" deviceset="R-NETZ@3" device="" value="33R"/>
-<part name="C27" library="rcl" deviceset="C-EU" device="C0603K" value="10nF"/>
-<part name="C24" library="rcl" deviceset="C-EU" device="C0603K" value="10nF"/>
-<part name="C25" library="rcl" deviceset="C-EU" device="C0603K" value="10nF"/>
-<part name="C26" library="rcl" deviceset="C-EU" device="C0603K" value="10nF"/>
-<part name="C30" library="rcl" deviceset="C-EU" device="C0603K" value="10nF"/>
-<part name="C28" library="rcl" deviceset="C-EU" device="C0603K" value="10nF"/>
-<part name="C29" library="rcl" deviceset="C-EU" device="C0603K" value="10nF"/>
-<part name="C31" library="rcl" deviceset="C-EU" device="C0603K" value="10nF"/>
+<part name="C27" library="rcl" deviceset="C-EU" device="C0603K" value="100nF"/>
+<part name="C24" library="rcl" deviceset="C-EU" device="C0603K" value="100nF"/>
+<part name="C25" library="rcl" deviceset="C-EU" device="C0603K" value="100nF"/>
+<part name="C26" library="rcl" deviceset="C-EU" device="C0603K" value="100nF"/>
+<part name="C30" library="rcl" deviceset="C-EU" device="C0603K" value="100nF"/>
+<part name="C28" library="rcl" deviceset="C-EU" device="C0603K" value="100nF"/>
+<part name="C29" library="rcl" deviceset="C-EU" device="C0603K" value="100nF"/>
+<part name="C31" library="rcl" deviceset="C-EU" device="C0603K" value="100nF"/>
 <part name="C19" library="rcl" deviceset="C-EU" device="C0603K" value="100nF"/>
 <part name="C20" library="rcl" deviceset="C-EU" device="C0603K" value="100nF"/>
@@
 <part name="R2" library="rcl" deviceset="R-EU_" device="R0603" value="4.7k"/>
 <part name="F1" library="rcl" deviceset="R-EU_" device="R2512" value="500mA"/>
-<part name="IC12" library="am29-memory" deviceset="AM29F010S" device=""/>
+<part name="IC12" library="am29-memory" deviceset="AM29F010S" device="" value="AM29F010S-10"/>
 <part name="IDE_ACT" library="con-molex" deviceset="22-?-02" device="05-7028"/>
 <part name="R1" library="rcl" deviceset="R-EU_" device="R0603" value="330"/>
 <part name="P+9" library="supply1" deviceset="VCC" device=""/>
-<part name="C39" library="rcl" deviceset="C-EU" device="C0805K" value="47µF"/>
+<part name="C39" library="rcl" deviceset="C-EU" device="C1206K" value="47uF"/>
 <part name="GND13" library="supply1" deviceset="GND" device=""/>
 <part name="C40" library="rcl" deviceset="C-EU" device="C0603K" value="100nF"/>
@@
 <part name="GND14" library="supply1" deviceset="GND" device=""/>
 <part name="P+10" library="supply1" deviceset="VCC" device=""/>
-<part name="IC13" library="xilinx_xc9572xl-tq100" deviceset="XC95288XL-TQ144" device=""/>
+<part name="IC13" library="xilinx_xc9572xl-tq100" deviceset="XC95288XL-TQ144" device="" value="XC95288XL-TQ144-10ns"/>
 <part name="C46" library="rcl" deviceset="C-EU" device="C0603K" value="100nF"/>
 <part name="C47" library="rcl" deviceset="C-EU" device="C0603K" value="100nF"/>
@@
 <part name="IC10" library="74xx-eu" deviceset="74*245" device="PW" technology="HCT" value="74HCT245PW"/>
 <part name="IC15" library="74xx-eu" deviceset="74*245" device="PW" technology="HCT" value="74HCT245PW"/>
-<part name="X1" library="SMD-Crystal" deviceset="CSX-750FC" device="FC(5V)"/>
-<part name="C43" library="rcl" deviceset="C-EU" device="C0603K"/>
+<part name="X1" library="SMD-Crystal" deviceset="CSX-750FC" device="FC(5V)" value="16,66MHz / 3.3V"/>
+<part name="C43" library="rcl" deviceset="C-EU" device="C0603K" value="100nF"/>
 <part name="+3V12" library="supply1" deviceset="+3V3" device=""/>
 <part name="GND39" library="supply1" deviceset="GND" device=""/>
-<part name="C44" library="rcl" deviceset="C-EU" device="C0603K"/>
-<part name="FB1" library="rcl" deviceset="R-EU_" device="R0603" value="100Ohm@100MHz"/>
+<part name="C44" library="rcl" deviceset="C-EU" device="C0603K" value="100nF"/>
+<part name="FB1" library="rcl" deviceset="R-EU_" device="R0603" value="120Ohm@100MHz 0.5A"/>
 <part name="R15" library="rcl" deviceset="R-EU_" device="R0603" value="33"/>
 <part name="R17" library="rcl" deviceset="R-EU_" device="R0603" value="33"/>

Commit message: Improved layout
Parts:
- added R3, R4: n.b., rcl:R-EU_R0603
- C44: value 100nF -> n.b.
- FB1: value 120Ohm@100MHz 0.5A -> n.b.
- IC14: value ICS570B -> ICS570A
- IC5: value LD117AS33TR -> LD117ADT33TR; device v-reg:LD117AS33TR -> v-reg:LD117ADT33TR
- R15: value 33 -> n.b.
- X1: value 16,66MHz / 3.3V -> n.b.
Connections:
- net +5V: no longer R12.2, R13.2
- net GND: now also R3.1, R4.1
- net S0: now also R4.2
- net S1: now also R3.2
- net VCC_IC14: now also R12.2, R13.2
Other:
- note added: "R3/R4 are populated with 4k7 for a 570B"
- moved on the sheet: C43, IC14, IC14G$2, R10, R11, SJ1, SJ2
